File: pnp/pcb/mobo/limit_switches.kicad_sch (KiCad schematic)
At the start: 12 parts, among them J2 X_LIMIT, J3 Y_LIMIT, J4 Z_LIMIT, J5 L_LIMIT, J6 R_LIMIT, J7 A_LIMIT

Commit message: tweak PN of mobo
Parts:
- JP25, JP26, JP29, JP30, JP31, JP32: LCSC (none) -> DNP
Changed lines of the file:
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@@
+      (effects (font (size 1.27 1.27)) hide)
+    )
+    (property "LCSC" "DNP" (at 189.23 86.36 0)
       (effects (font (size 1.27 1.27)) hide)
     )
@@
       (effects (font (size 1.27 1.27)) hide)
     )
+    (property "LCSC" "DNP" (at 189.23 121.92 0)
+      (effects (font (size 1.27 1.27)) hide)
+    )
     (pin "1")
     (pin "2")
@@
       (effects (font (size 1.27 1.27)) hide)
     )
+    (property "LCSC" "DNP" (at 189.23 68.58 0)
+      (effects (font (size 1.27 1.27)) hide)
+    )
     (pin "1")
     (pin "2")
@@
       (effects (font (size 1.27 1.27)) hide)
     )
+    (property "LCSC" "DNP" (at 189.23 105.41 0)
+      (effects (font (size 1.27 1.27)) hide)
+    )
     (pin "1")
     (pin "2")
@@
       (effects (font (size 1.27 1.27)) hide)
     )
+    (property "LCSC" "DNP" (at 189.23 156.21 0)
+      (effects (font (size 1.27 1.27)) hide)
+    )
     (pin "1")
     (pin "2")
@@
       (effects (font (size 1.27 1.27)) hide)
     )
+    (property "LCSC" "DNP" (at 189.23 139.7 0)
+      (effects (font (size 1.27 1.27)) hide)
+    )
