File: pnp/pcb/mobo/miscellaneous.kicad_sch (KiCad schematic)
At the start: 10 parts

Commit message: tweak PN of mobo
Parts:
- FID1, FID2, FID3, FID4, FID5, FID6, H5, H6, H7, H8: LCSC (none) -> DNP
Changed lines of the file:
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@@
+      (effects (font (size 1.27 1.27)) hide)
+    )
+    (property "LCSC" "DNP" (at 134.62 96.52 0)
       (effects (font (size 1.27 1.27)) hide)
     )
@@
       (effects (font (size 1.27 1.27)) hide)
     )
+    (property "LCSC" "DNP" (at 134.62 106.68 0)
+      (effects (font (size 1.27 1.27)) hide)
+    )
     (instances
       (project "mobo"
@@
     )
     (property "Datasheet" "" (at 134.62 101.6 0)
+      (effects (font (size 1.27 1.27)) hide)
+    )
+    (property "LCSC" "DNP" (at 134.62 101.6 0)
       (effects (font (size 1.27 1.27)) hide)
     )
@@
       (effects (font (size 1.27 1.27)) hide)
     )
+    (property "LCSC" "DNP" (at 163.83 106.68 0)
+      (effects (font (size 1.27 1.27)) hide)
+    )
     (pin "1")
     (instances
@@
       (effects (font (size 1.27 1.27)) hide)
     )
+    (property "LCSC" "DNP" (at 163.83 124.46 0)
+      (effects (font (size 1.27 1.27)) hide)
+    )
     (pin "1")
     (instances
@@
       (effects (font (size 1.27 1.27)) hide)
     )
+    (property "LCSC" "DNP" (at 134.62 118.11 0)
+      (effects (font (size 1.27 1.27)) hide)
+    )
     (instances
       (project "mobo"
@@
       (effects (font (size 1.27 1.27)) hide)
     )
+    (property "LCSC" "DNP" (at 163.83 97.79 0)
+      (effects (font (size 1.27 1.27)) hide)
+    )
     (pin "1")
     (instances
@@
       (effects (font (size 1.27 1.27)) hide)
     )
+    (property "LCSC" "DNP" (at 134.62 128.27 0)
+      (effects (font (size 1.27 1.27)) hide)
+    )
     (instances
       (project "mobo"
@@
       (effects (font (size 1.27 1.27)) hide)
     )
+    (property "LCSC" "DNP" (at 163.83 115.57 0)
+      (effects (font (size 1.27 1.27)) hide)
+    )
     (pin "1")
     (instances
@@
       (effects (font (size 1.27 1.27)) hide)
     )
+    (property "LCSC" "DNP" (at 134.62 123.19 0)
+      (effects (font (size 1.27 1.27)) hide)
+    )
