File: pnp/pcb/mobo/mosfet.kicad_sch (KiCad schematic)
At the start: 5 parts, among them J22 Mosfet, Q1 AO3400A

Commit message: tweak PN of mobo
Parts:
- R30: JLCPCB C4360 -> C17414; LCSC C139879 -> C115295
Changed lines of the file:
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@@
       (effects (font (size 1.27 1.27)) hide)
     )
-    (property "JLCPCB" "C4360" (at 140.97 109.22 0)
+    (property "JLCPCB" "C17414" (at 140.97 109.22 0)
       (effects (font (size 1.27 1.27)) hide)
     )
-    (property "LCSC" "C139879" (at 140.97 109.22 0)
+    (property "LCSC" "C115295" (at 140.97 109.22 0)
       (effects (font (size 1.27 1.27)) hide)
     )
