File: pnp/pcb/mobo/servos.kicad_sch (KiCad schematic)
At the start: 3 parts, among them J15 SERVO1, J16 SERVO2, U7 SN74LVC2G34

Commit message: tweak PN of mobo
Parts:
- U7: LCSC (none) -> C347589
Changed lines of the file:
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@@
+      (effects (font (size 1.27 1.27)) hide)
+    )
+    (property "LCSC" "C347589" (at 111.76 106.045 0)
       (effects (font (size 1.27 1.27)) hide)
     )
