File: pnp/pcb/mobo/usb.kicad_sch (KiCad schematic)
At the start: 4 parts, among them J9 USB_B, U8 SRV05-4

Commit message: tweak PN of mobo
Parts:
- J9: LCSC (none) -> C720549
- TP1, TP2: LCSC (none) -> DNP
- U8: LCSC (none) -> C2972082
Changed lines of the file:
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@@
+      (effects (font (size 1.27 1.27)) hide)
+    )
+    (property "LCSC" "DNP" (at 87.63 118.11 0)
       (effects (font (size 1.27 1.27)) hide)
     )
@@
     )
     (property "Datasheet" "~" (at 87.63 129.54 0)
+      (effects (font (size 1.27 1.27)) hide)
+    )
+    (property "LCSC" "DNP" (at 87.63 124.46 0)
       (effects (font (size 1.27 1.27)) hide)
     )
@@
     )
     (property "Notes" "USB TVS" (at 144.145 79.375 0)
+      (effects (font (size 1.27 1.27)) hide)
+    )
+    (property "LCSC" "C2972082" (at 144.145 79.375 0)
       (effects (font (size 1.27 1.27)) hide)
     )
@@
       (effects (font (size 1.27 1.27)) hide)
     )
+    (property "LCSC" "C720549" (at 77.47 75.565 0)
+      (effects (font (size 1.27 1.27)) hide)
+    )
